File: AppRelay/AppRelay.sch (KiCad schematic (older format))
At the start: 14 parts, among them P1 CONN_01X04, P2 CONN_01X01, P3 CONN_01X01, Q1 Q_NPN_BEC, Q2 Q_NPN_BEC, X1 RELAY_SPST

Commit message: Added suggested NPN driver part numbers.
Parts:
- Q1, Q2: MFRPN (none) -> MMBT3904
- X1: MFRPN (none) -> G6BU-1114P-US-DC12
Changed lines of the file:
@@
 F 2 "pwr_relay:G6BU-1114P-US-DC12" H 7100 4250 60  0001 C CNN
 F 3 "http://www.digikey.com/product-detail/en/omron-electronics-inc-emc-div/G6BU-1114P-US-DC12/Z3702-ND/369136" H 7100 4250 60  0001 C CNN
+F 4 "G6BU-1114P-US-DC12" H 7100 4250 60  0001 C CNN "MFRPN"
 	1    7100 4250
 	1    0    0    -1
@@
 F 2 "TO_SOT_Packages_SMD:SOT-23" H 3800 5100 50  0001 C CNN
 F 3 "" H 3600 5000 50  0000 C CNN
+F 4 "MMBT3904" H 3600 5000 60  0001 C CNN "MFRPN"
 	1    3600 5000
 	1    0    0    -1
@@
 F 2 "TO_SOT_Packages_SMD:SOT-23" H 5000 4750 50  0001 C CNN
 F 3 "" H 4800 4650 50  0000 C CNN
+F 4 "MMBT3904" H 4800 4650 60  0001 C CNN "MFRPN"
 	1    4800 4650
 	1    0    0    -1
